Commit message: Updated urdf to reference new name for description pkg

File: urdf/pioneer3dx.xacro (robot description, xacro)
@@ -3,7 +3,7 @@
 <!-- Git repository at https://github.com/allenh1/p2os -->
 <robot name="pioneer3dx" xmlns:xacro="http://ros.org/wiki/xacro">
-  <xacro:include filename="$(find pioneer_description)/urdf/pioneer3dx_wheel.xacro"/>
-  <xacro:include filename="$(find pioneer_description)/urdf/materials.xacro" />
-  <xacro:include filename="$(find pioneer_description)/urdf/pioneer.gazebo" />
+  <xacro:include filename="$(find pioneer_3dx_description)/urdf/pioneer3dx_wheel.xacro"/>
+  <xacro:include filename="$(find pioneer_3dx_description)/urdf/materials.xacro" />
+  <xacro:include filename="$(find pioneer_3dx_description)/urdf/pioneer.gazebo" />
 <!-- Base link to interface with gmapping and move_base -->
 	<link name="base_link"/>
@@ -15,8 +15,8 @@
   </joint>
   <link name="chassis">
-    <visual name="chassis_visual">
+    <visual name="chassis_visual">ea
       <origin xyz="0 0 0" rpy="0 0 0"/>
 			<geometry name="pioneer_geom">
-				<mesh filename="package://pioneer_description/meshes/p3dx_meshes/chassis.stl"/>
+				<mesh filename="file://$(find pioneer_3dx_description)/meshes/p3dx_meshes/chassis.stl"/>
 			</geometry>
 			<material name="ChassisRed"/>
@@ -25,5 +25,5 @@
 			<origin xyz="0 0 0" rpy="0 0 0"/>
 			<geometry>
-				<mesh filename="package://pioneer_description/meshes/p3dx_meshes/chassis.stl"/>
+				<mesh filename="file://$(find pioneer_3dx_description)/meshes/p3dx_meshes/chassis.stl"/>
 				<!--box size="0.43 0.277 0.17"/-->
 			</geometry>
@@ -54,5 +54,5 @@
 			<origin xyz="0 0 0" rpy="0 0 0"/>
 			<geometry name="top_geom">
-				<mesh filename="package://pioneer_description/meshes/p3dx_meshes/top.stl"/>
+				<mesh filename="file://$(find pioneer_3dx_description)/meshes/p3dx_meshes/top.stl"/>
 			</geometry>
 			<material name="TopBlack"/>
@@ -61,5 +61,5 @@
 			<origin xyz="0 0 0" rpy="0 0 0"/>
 			<geometry>
-				<mesh filename="package://pioneer_description/meshes/p3dx_meshes/top.stl"/>
+				<mesh filename="file://$(find pioneer_3dx_description)/meshes/p3dx_meshes/top.stl"/>
 				<!--box size="0.44 0.38 0.005"/-->
 			</geometry>
@@ -86,5 +86,5 @@
 		  <origin xyz="0 0 0" rpy="0 0 0"/>
 		  <geometry name="pioneer_geom">
-			  <mesh filename="package://pioneer_description/meshes/p3dx_meshes/swivel.stl"/>
+			  <mesh filename="file://$(find pioneer_3dx_description)/meshes/p3dx_meshes/swivel.stl"/>
 		  </geometry>
 		  <material name="swivel"/>
@@ -93,5 +93,5 @@
 		  <origin xyz="0 0 0" rpy="0 0 0"/>
 		  <geometry>
-			  <mesh filename="package://pioneer_description/meshes/p3dx_meshes/swivel.stl"/>
+			  <mesh filename="file://$(find pioneer_3dx_description)/meshes/p3dx_meshes/swivel.stl"/>
 		  </geometry>
 	  </collision>
@@ -108,5 +108,5 @@
 		  <origin xyz="0 0 0" rpy="0 0 0"/>
 		  <geometry name="pioneer_geom">
-			  <mesh filename="package://pioneer_description/meshes/p3dx_meshes/center_hubcap.stl"/>
+			  <mesh filename="file://$(find pioneer_3dx_description)/meshes/p3dx_meshes/center_hubcap.stl"/>
 		  </geometry>
 		  <material name="HubcapGrey"/>
@@ -115,5 +115,5 @@
 		  <origin xyz="0 0 0" rpy="0 0 0"/>
 		  <geometry>
-			  <mesh filename="package://pioneer_description/meshes/p3dx_meshes/center_hubcap.stl"/>
+			  <mesh filename="file://$(find pioneer_3dx_description)/meshes/p3dx_meshes/center_hubcap.stl"/>
 		  </geometry>
 	  </collision>
@@ -138,5 +138,5 @@
 		  <origin xyz="0 0 0" rpy="0 0 0"/>
 		  <geometry name="pioneer_geom">
-			  <mesh filename="package://pioneer_description/meshes/p3dx_meshes/center_wheel.stl"/>
+			  <mesh filename="file://$(find pioneer_3dx_description)/meshes/p3dx_meshes/center_wheel.stl"/>
 		  </geometry>
 		  <material name="WheelBlack"/>
@@ -145,5 +145,5 @@
 		  <origin xyz="0 0 0" rpy="0 0 0"/>
 		  <geometry>
-		    <mesh filename="package://pioneer_description/meshes/p3dx_meshes/center_wheel.stl"/>
+		    <mesh filename="file://$(find pioneer_3dx_description)/meshes/p3dx_meshes/center_wheel.stl"/>
 			  <!--<cylinder radius="0.0375" length="0.03"/>-->
 		  </geometry>
@@ -175,5 +175,5 @@
 			<origin xyz="0 0 0" rpy="0 0 0"/>
 			<geometry>
-				<mesh filename="package://pioneer_description/meshes/p3dx_meshes/left_wheel.stl"/>
+				<mesh filename="file://$(find pioneer_3dx_description)/meshes/p3dx_meshes/left_wheel.stl"/>
 			</geometry>
 			<material name="WheelBlack"/>
@@ -182,5 +182,5 @@
 			<origin xyz="0 0 0" rpy="0 0 0"/>
 			<geometry>
-			  <mesh filename="package://pioneer_description/meshes/p3dx_meshes/left_wheel.stl"/>
+			  <mesh filename="file://$(find pioneer_3dx_description)/meshes/p3dx_meshes/left_wheel.stl"/>
 				<!--<cylinder radius="0.092" length="0.04"/>-->
 			</geometry>
@@ -196,5 +196,5 @@
 			<origin xyz="0 0 0" rpy="0 0 0"/>
 			<geometry>
-				<mesh filename="package://pioneer_description/meshes/p3dx_meshes/left_hubcap.stl"/>
+				<mesh filename="file://$(find pioneer_3dx_description)/meshes/p3dx_meshes/left_hubcap.stl"/>
 			</geometry>
 			<material name="HubcapYellow"/>
@@ -203,5 +203,5 @@
 			<origin xyz="0 0 0" rpy="0 0 0"/>
 			<geometry>
-				<mesh filename="package://pioneer_description/meshes/p3dx_meshes/left_hubcap.stl"/>
+				<mesh filename="file://$(find pioneer_3dx_description)/meshes/p3dx_meshes/left_hubcap.stl"/>
 			</geometry>
 		</collision>
@@ -227,5 +227,5 @@
 			<origin xyz="0 0 0" rpy="0 0 0"/>
 			<geometry>
-				<mesh filename="package://pioneer_description/meshes/p3dx_meshes/right_wheel.stl"/>
+				<mesh filename="file://$(find pioneer_3dx_description)/meshes/p3dx_meshes/right_wheel.stl"/>
 			</geometry>
 			<material name="WheelBlack"/>
@@ -234,5 +234,5 @@
 			<origin xyz="0 0 0" rpy="0 0 0"/>
 			<geometry>
-			  <mesh filename="package://pioneer_description/meshes/p3dx_meshes/right_wheel.stl"/>
+			  <mesh filename="file://$(find pioneer_3dx_description)/meshes/p3dx_meshes/right_wheel.stl"/>
 				<!--<cylinder radius="0.092" length="0.04"/>-->
 			</geometry>
@@ -248,5 +248,5 @@
 			<origin xyz="0 0 0" rpy="0 0 0"/>
 			<geometry>
-				<mesh filename="package://pioneer_description/meshes/p3dx_meshes/right_hubcap.stl"/>
+				<mesh filename="file://$(find pioneer_3dx_description)/meshes/p3dx_meshes/right_hubcap.stl"/>
 			</geometry>
 			<material name="HubcapYellow"/>
@@ -255,5 +255,5 @@
 			<origin xyz="0 0 0" rpy="0 0 0"/>
 			<geometry>
-				<mesh filename="package://pioneer_description/meshes/p3dx_meshes/right_hubcap.stl"/>
+				<mesh filename="file://$(find pioneer_3dx_description)/meshes/p3dx_meshes/right_hubcap.stl"/>
 			</geometry>
 		</collision>
@@ -270,5 +270,5 @@
 			<origin xyz="0 0 0" rpy="0 0 0"/>
 			<geometry name="pioneer_geom">
-				<mesh filename="package://pioneer_description/meshes/p3dx_meshes/front_sonar.stl"/>
+				<mesh filename="file://$(find pioneer_3dx_description)/meshes/p3dx_meshes/front_sonar.stl"/>
 			</geometry>
 			<material name="SonarYellow"/>
@@ -277,5 +277,5 @@
 			<origin xyz="0 0 0" rpy="0 0 0"/>
 			<geometry>
-				<mesh filename="package://pioneer_description/meshes/p3dx_meshes/front_sonar.stl"/>
+				<mesh filename="file://$(find pioneer_3dx_description)/meshes/p3dx_meshes/front_sonar.stl"/>
 			</geometry>
 		</collision>
@@ -296,5 +296,5 @@
 			<origin xyz="0 0 0" rpy="0 0 0"/>
 			<geometry name="pioneer_geom">
-				<mesh filename="package://pioneer_description/meshes/p3dx_meshes/back_sonar.stl"/>
+				<mesh filename="file://$(find pioneer_3dx_description)/meshes/p3dx_meshes/back_sonar.stl"/>
 			</geometry>
 			<material name="SonarYellow"/>
@@ -303,5 +303,5 @@
 			<origin xyz="0 0 0" rpy="0 0 0"/>
 			<geometry>
-				<mesh filename="package://pioneer_description/meshes/p3dx_meshes/back_sonar.stl"/>
+				<mesh filename="file://$(find pioneer_3dx_description)/meshes/p3dx_meshes/back_sonar.stl"/>
 			</geometry>
 		</collision>
@@ -322,5 +322,5 @@
       <origin xyz="0 0 0" rpy="0 0 0"/>
       <geometry>
-        <mesh filename="package://pioneer_description/meshes/hokuyo.dae"/>
+        <mesh filename="file://$(find pioneer_3dx_description)/meshes/hokuyo.dae"/>
 	      <!--box size="0.05 0.05 0.071"/-->
       </geometry>
@@ -329,5 +329,5 @@
       <origin xyz="0 0 0" rpy="0 0 0"/>
       <geometry>
-        <mesh filename="package://pioneer_description/meshes/hokuyo.dae"/>
+        <mesh filename="file://$(find pioneer_3dx_description)/meshes/hokuyo.dae"/>
       </geometry>
     </visual>

File: urdf/pioneer3dx_wheel.xacro (robot description, xacro)
@@ -21,5 +21,5 @@
       <origin xyz="0 0 0" rpy="0 0 0"/>
       <geometry name="pioneer_geom">
-        <mesh filename="package://pioneer_description/meshes/p3dx_meshes/${suffix}_wheel.stl"/>
+        <mesh filename="($find pioneer_3dx_description)/meshes/p3dx_meshes/${suffix}_wheel.stl"/>
       </geometry>
       <material name="WheelBlack">
@@ -30,5 +30,5 @@
       <origin xyz="0 0 0" rpy="${-3.1415927/2} 0 0"/>
       <geometry>
-        <!--<mesh filename="package://pioneer_description/meshes/p3dx_meshes/${suffix}_wheel.stl"/>-->
+        <!--<mesh filename="($find pioneer_3dx_description)/meshes/p3dx_meshes/${suffix}_wheel.stl"/>-->
         <cylinder radius="0.09" length="0.01"/>
       </geometry>
@@ -51,5 +51,5 @@
     <origin xyz="0 0 0" rpy="0 0 0"/>
     <geometry name="pioneer_geom">
-      <mesh filename="package://pioneer_description/meshes/p3dx_meshes/${suffix}_hubcap.stl"/>
+      <mesh filename="($find pioneer_3dx_description)/meshes/p3dx_meshes/${suffix}_hubcap.stl"/>
     </geometry>
     <material name="HubcapYellow">
